File: BitPad/BitPad/BitPad.kicad_pcb (KiCad board)
At the start: 2 copper layers, 10 parts, among them SW1 SW_Push, SW2 SW_Push, SW3 SW_Push, SW4 SW_Push, SW5 SW_MEC_5E, U1 MOUDLE-SEEEDUINO-XIAO

Commit message: updated the kicad files
Parts:
- D1, D2, D3, D4: footprint Diode_SMD:D_SMA -> Diode_SMD:D_0201_0603Metric
- SW5: value SW_MEC_5E -> SW_Push; footprint Button_Switch_Keyboard:SW_Cherry_MX_1.00u_PCB -> Button_Switch_THT:SW_TH_Tactile_Omron_B3F-100x
- moved SW5 71.9 mm to (124.5, 62.5)
- moved D4 40.6 mm to (144.2, 130.5)
- moved D2 40.5 mm to (144.0, 100.5)
- moved D1 40.0 mm to (143.8, 84.0)
- moved D3 40.0 mm to (143.7, 115.0)
- moved SW2 13.8 mm to (130.6, 95.6)
- moved SW3 13.8 mm to (130.6, 110.6)
- moved SW4 13.8 mm to (130.6, 125.7)
- moved U1 13.8 mm to (128.6, 84.1), turned to 90 degrees
- moved SW1 13.2 mm to (130.0, 80.0)
Connections:
- D1 pad 1: Net-(D1-K) -> GND
- D1 pad 2: GND -> Net-(D1-A)
- D2 pad 1: Net-(D2-K) -> GND
- D2 pad 2: GND -> Net-(D2-A)
- D3 pad 1: Net-(D3-K) -> GND
- D3 pad 2: GND -> Net-(D3-A)
- D4 pad 1: Net-(D4-K) -> GND
- D4 pad 2: GND -> Net-(D4-A)
- SW1 pad 2: Net-(D1-K) -> GND
- SW2 pad 2: Net-(D2-K) -> GND
- SW3 pad 2: Net-(D3-K) -> GND
- SW4 pad 2: Net-(D4-K) -> GND
- SW5 pad 1: Net-(D1-K) -> GND
- SW5 pad 2: Net-(D2-K) -> Net-(U1-PB08_A6_D6_TX)
- U1 pad 2: unconnected-(U1-PA4_A1_D1-Pad2) -> Net-(D1-A)
- U1 pad 3: unconnected-(U1-PA10_A2_D2-Pad3) -> Net-(D2-A)
- U1 pad 4: unconnected-(U1-PA11_A3_D3-Pad4) -> Net-(D3-A)
- U1 pad 5: unconnected-(U1-PA8_A4_D4_SDA-Pad5) -> Net-(D4-A)
- U1 pad 7: unconnected-(U1-PB08_A6_D6_TX-Pad7) -> Net-(U1-PB08_A6_D6_TX)
